Commit message: Adds example code, increases max episode steps for rocketlander

File: brs_data/martlet9/martlet9.urdf (robot description, URDF)
Before this commit: robot martlet9, 11 links, 10 joints
Links:
- link base: mass 200000 -> 400000
- link thruster: mass 175000 -> 75000
- link thruster_casing: mass 200000 -> 100000

File: brs_data/martlet9/martlet9.urdf.xacro (robot description, xacro)
@@ -3,5 +3,5 @@
   <xacro:property name="base_height" value="70"/>
   <xacro:property name="base_radius" value="1.85"/>
-  <xacro:property name="base_mass" value="200000"/>
+  <xacro:property name="base_mass" value="400000"/>
   <xacro:property name="base_inertia_radial"
                   value="${base_mass * (0.25 * base_radius * base_radius + base_height * base_height / 12)}"/>
@@ -15,8 +15,8 @@
   <xacro:property name="steer1_wheel_z" value="20"/>
   <xacro:property name="steer_gun_x" value="${steer_wheel_radius + steer_gun_length / 2}"/>
-  <xacro:property name="thruster_casing_mass" value="200000"/>
+  <xacro:property name="thruster_casing_mass" value="100000"/>
   <xacro:property name="thruster_casing_r" value="1.7"/>
   <xacro:property name="thruster_casing_l" value="8"/>
-  <xacro:property name="thruster_mass" value="175000"/>
+  <xacro:property name="thruster_mass" value="75000"/>
   <xacro:property name="thruster_r" value="1.2"/>
   <xacro:property name="thruster_l" value="4"/>

Commit message: Adds smoke effects

File: brs_data/martlet9/martlet9.urdf (robot description, URDF)
Before this commit: robot martlet9, 11 links, 10 joints
Links:
- added link steer1_smoke, mass 0; visual cylinder length=5 radius=0.225
- added link thruster_fire, mass 0; visual cylinder length=5 radius=1.08
Joints:
- added joint steer1_gun_to_smoke: type fixed, parent steer1_gun, child steer1_smoke, origin xyz=3.5 0 0
- added joint thruster_to_fire: type fixed, parent thruster, child thruster_fire, origin xyz=0 0 -5.0

File: brs_data/martlet9/martlet9.urdf.xacro (robot description, xacro)
@@ -18,4 +18,5 @@
   <xacro:property name="thruster_casing_r" value="1.7"/>
   <xacro:property name="thruster_casing_l" value="8"/>
+  <xacro:property name="thruster_casing_z" value="-32"/>
   <xacro:property name="thruster_mass" value="75000"/>
   <xacro:property name="thruster_r" value="1.2"/>
@@ -29,4 +30,10 @@
   <xacro:property name="thruster_inertia"
                   value="${thruster_mass * 0.5 * thruster_r * thruster_r}"/>
+  <xacro:property name="thruster_fire_r" value="${thruster_r * 0.9}"/>
+  <xacro:property name="thruster_fire_l" value="5"/>
+  <xacro:property name="thruster_fire_z" value="${-0.5 - thruster_l/2 - thruster_fire_l/2}"/>
+  <xacro:property name="steering_smoke_r" value="${steer_gun_size * 0.9}"/>
+  <xacro:property name="steering_smoke_l" value="5"/>
+  <xacro:property name="steering_smoke_x" value="${0.5 + steer_gun_length / 2 + steering_smoke_l / 2}"/>
   <material name="white">
     <color rgba="1 1 1 1"/>
@@ -38,4 +45,10 @@
     <color rgba="0.4 0.4 0.4 0.9"/>
   </material>
+  <material name="thruster_fire_mat">
+    <color rgba="1.0 1.0 0.3 0.0"/>
+  </material>
+  <material name="steering_smoke_mat">
+    <color rgba="0.3 0.3 0.3 0.0"/>
+  </material>
   <link name="base">
     <visual>
@@ -89,4 +102,16 @@
     </inertial>
   </link>
+  <link name="thruster_fire">
+    <visual>
+      <geometry>
+        <cylinder length="${thruster_fire_l}" radius="${thruster_fire_r}"/>
+      </geometry>
+      <material name="thruster_fire_mat"/>
+    </visual>
+    <inertial>
+      <mass value="0"/>
+      <inertia ixx="1" ixy="0" ixz="0" iyy="1" iyz="0" izz="1"/>
+    </inertial>
+  </link>
   <link name="steer1_wheel">
     <visual>
@@ -120,4 +145,17 @@
     <inertial>
       <mass value="${steer_gun_mass}"/>
+      <inertia ixx="1" ixy="0" ixz="0" iyy="1" iyz="0" izz="1"/>
+    </inertial>
+  </link>
+  <link name="steer1_smoke">
+    <visual>
+      <geometry>
+        <cylinder length="${steering_smoke_l}" radius="${steering_smoke_r}"/>
+      </geometry>
+      <origin rpy="0 1.57 0"/>
+      <material name="steering_smoke_mat"/>
+    </visual>
+    <inertial>
+      <mass value="0"/>
       <inertia ixx="1" ixy="0" ixz="0" iyy="1" iyz="0" izz="1"/>
     </inertial>
@@ -249,5 +287,5 @@
     <parent link="base"/>
     <child link="thruster_casing"/>
-    <origin xyz="0 0 -32"/>
+    <origin xyz="0 0 ${thruster_casing_z}"/>
   </joint>
   <joint name="thruster_casing_to_thruster" type="fixed">
@@ -256,4 +294,9 @@
     <origin xyz="0 0 -3"/>
   </joint>
+  <joint name="thruster_to_fire" type="fixed">
+    <parent link="thruster"/>
+    <child link="thruster_fire"/>
+    <origin xyz="0 0 ${thruster_fire_z}"/>
+  </joint>
   <joint name="base_to_steer1_wheel" type="continuous">
     <parent link="base"/>
@@ -267,4 +310,9 @@
     <origin xyz="${steer_gun_x} 0 0"/>
   </joint>
+  <joint name="steer1_gun_to_smoke" type="fixed">
+    <parent link="steer1_gun"/>
+    <child link="steer1_smoke"/>
+    <origin xyz="${steering_smoke_x} 0 0"/>
+  </joint>
   <joint name="leg1_to_ball" type="fixed">
     <parent link="leg1"/>
